File: lora-calculator_jlcpcb.kicad_pcb (KiCad board)
At the start: 2 copper layers, 190 x 175 mm, 84 parts, among them J1 USB-C, J2 PinHeader_1x04_P2.54mm_Vertic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, J3 LipoCable, SW1 SW_Push, SW10 SW_Push, SW11 SW_Push, SW12 SW_Push, SW13 SW_Push, SW14 SW_Push, SW15 SW_Push, SW16 SW_Push, SW17 SW_Push, SW18 SW_Push, SW19 SW_Push, SW2 SW_Push, SW20 SW_Push, SW21 SW_Push, SW22 SW_Push, SW23 SW_Push, SW24 SW_Push, SW25 SW_Push, SW26 SW_Push, SW27 SW_Push, SW28 SW_Push, SW29 SW_Push, SW3 SW_Push, SW30 SW_Push, SW31 SW_SPDT, SW4 SW_Push, SW5 SW_Push, SW6 SW_Push, SW7 SW_Push, SW8 SW_Push, SW9 SW_Push, U1 MCP23017x-x-SO, U3 MCP73831-2-OT, U4 ESP32-C3-WROOM-02U, U5 AP2112K-3.3

Commit message: Update KiCad PCB layout
Co-Authored-By: Claude Haiku 5.5 <noreply@anthropic.com>
Parts:
- moved U1 226.4 mm to (216.5, 27.5)
- moved U3 226.4 mm to (231.5, 27.5)
- moved U4 226.4 mm to (246.5, 27.5)
- moved U5 226.4 mm to (261.5, 27.5)
- moved J3 142.0 mm to (100.9, -36.7)
- moved R1 142.0 mm to (115.9, -36.7)
- moved R10 142.0 mm to (220.9, -36.7)
- moved R2 142.0 mm to (130.9, -36.7)
- moved R3 142.0 mm to (145.9, -36.7)
- moved R6 142.0 mm to (160.9, -36.7)
- moved R7 142.0 mm to (175.9, -36.7)
- moved R8 142.0 mm to (190.9, -36.7)
- moved R9 142.0 mm to (205.9, -36.7)
- moved C1 130.6 mm to (130.6, -49.5)
- moved C10 130.6 mm to (235.6, -49.5)
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Changed lines of the file:
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@@
 		(tags "tact sw push 6mm silicone rubber")
 		(property "Reference" "SW1"
-			(at 0 -4.064 0)
+			(at 47.45 -90.624 0)
 			(layer "F.SilkS")
 			(effects
@@
 		)
 		(fp_text user "REF**"
-			(at 0 -4.064 0)
+			(at 47.45 -90.624 0)
 			(layer "F.SilkS")
 			(effects
@@
 	(footprint "SOT-23-5"
 		(layer "F.Cu")
-		(at 65 140)
+		(at 261.53 27.52)
 		(descr "SOT, 5 Pin (JEDEC MO-178 Var AA https://www.jedec.org/document_search?search_api_views_fulltext=MO-178)")
 		(tags "SOT TO_SOT_SMD")
@@
 	(footprint "SOIC-28W_7.5x17.9mm_P1.27mm"
 		(layer "F.Cu")
-		(at 20 140)
+		(at 216.53 27.52)
 		(descr "SOIC, 28 Pin (JEDEC MS-013AE, https://www.analog.com/media/en/package-pcb-resources/package/35833120341221rw_28.pdf)")
 		(tags "SOIC SO")
@@
 	(footprint "D_SOD-123"
 		(layer "F.Cu")
-		(at 140 20)
+		(at 20.38 25.54)
 		(descr "SOD-123")
 		(tags "SOD-123")
@@
 	(footprint "C_0805_2012Metric"
 		(layer "F.Cu")
-		(at 20 20)
+		(at 130.57 -49.54)
 		(descr "Capacitor SMD 0805 (2012 Metric), square (rectangular) end terminal, IPC-7351 nominal, (Body size source: IPC-SM-782 page 76, https://www.pcb-3d.com/wordpress/wp-content/uploads/ipc-sm-782a_amendment_1_and_2.pdf, https://docs.google.com/spreadsheets/d/1BsfQQcO9C6DZCsRaXUlFlo91Tg2WpOkGARC1WS5S8t0/edit?usp=sharing)")
 		(tags "capacitor")
@@
 	(footprint "ESP32-C3-WROOM-02U"
 		(layer "F.Cu")
-		(at 50 140)
+		(at 246.53 27.52)
 		(descr "RF Module, ESP32-C3 WROOM-02 , Wi-Fi and Bluetooth, BLE, external antenna, https://www.espressif.com/sites/default/files/documentation/esp32-c3-wroom-02_datasheet_en.pdf")
 		(tags "ESP32-C3 WROOM-02 espressif")
@@
 	(footprint "USB_C_Receptacle_HRO_TYPE-C-31-M-12"
 		(layer "F.Cu")
-		(at 140 65)
+		(at 187.45 -21.56)
 		(descr "USB Type-C receptacle for USB 2.0 and PD, http://www.krhro.com/uploads/soft/180320/1-1P320120243.pdf")
 		(tags "usb usb-c 2.0 pd")
@@
 	(footprint "R_0603_1608Metric"
 		(layer "F.Cu")
-		(at 35 80)
+		(at 115.945 -36.7)
 		(descr "Resistor SMD 0603 (1608 Metric), square (rectangular) end terminal, IPC-7351 nominal, (Body size source: IPC-SM-782 page 72, https://www.pcb-3d.com/wordpress/wp-content/uploads/ipc-sm-782a_amendment_1_and_2.pdf)")
 		(tags "resistor")
@@
 	(footprint "C_0603_1608Metric"
 		(layer "F.Cu")
-		(at 50 20)
+		(at 160.57 -49.54)
 		(descr "Capacitor SMD 0603 (1608 Metric), square (rectangular) end terminal, IPC-7351 nominal, (Body size source: IPC-SM-782 page 76, https://www.pcb-3d.com/wordpress/wp-content/uploads/ipc-sm-782a_amendment_1_and_2.pdf)")
 		(tags "capacitor")
@@
 	(footprint "C_0603_1608Metric"
 		(layer "F.Cu")
-		(at 125 20)
+		(at 235.57 -49.54)
 		(descr "Capacitor SMD 0603 (1608 Metric), square (rectangular) end terminal, IPC-7351 nominal, (Body size source: IPC-SM-782 page 76, https://www.pcb-3d.com/wordpress/wp-content/uploads/ipc-sm-782a_amendment_1_and_2.pdf)")
 		(tags "capacitor")
@@
 	(footprint "R_0603_1608Metric"
 		(layer "F.Cu")
-		(at 80 80)
+		(at 160.945 -36.7)
 		(descr "Resistor SMD 0603 (1608 Metric), square (rectangular) end terminal, IPC-7351 nominal, (Body size source: IPC-SM-782 page 72, https://www.pcb-3d.com/wordpress/wp-content/uploads/ipc-sm-782a_amendment_1_and_2.pdf)")
 		(tags "resistor")
@@
 	(footprint "C_0603_1608Metric"
 		(layer "F.Cu")
-		(at 65 20)
+		(at 175.57 -49.54)
 		(descr "Capacitor SMD 0603 (1608 Metric), square (rectangular) end terminal, IPC-7351 nominal, (Body size source: IPC-SM-782 page 76, https://www.pcb-3d.com/wordpress/wp-content/uploads/ipc-sm-782a_amendment_1_and_2.pdf)")
 		(tags "capacitor")
@@
 	(footprint "R_0603_1608Metric"
 		(layer "F.Cu")
-		(at 140 80)
+		(at 220.945 -36.7)
 		(descr "Resistor SMD 0603 (1608 Metric), square (rectangular) end terminal, IPC-7351 nominal, (Body size source: IPC-SM-782 page 72, https://www.pcb-3d.com/wordpress/wp-content/uploads/ipc-sm-782a_amendment_1_and_2.pdf)")
 		(tags "resistor")
@@
 	(footprint "C_0805_2012Metric"
 		(layer "F.Cu")
-		(at 80 20)
+		(at 190.57 -49.54)
 		(descr "Capacitor SMD 0805 (2012 Metric), square (rectangular) end terminal, IPC-7351 nominal, (Body size source: IPC-SM-782 page 76, https://www.pcb-3d.com/wordpress/wp-content/uploads/ipc-sm-782a_amendment_1_and_2.pdf, https://docs.google.com/spreadsheets/d/1BsfQQcO9C6DZCsRaXUlFlo91Tg2WpOkGARC1WS5S8t0/edit?usp=sharing)")
 		(tags "capacitor")
@@
 	(footprint "R_0603_1608Metric"
 		(layer "F.Cu")
-		(at 110 80)
+		(at 190.945 -36.7)
 		(descr "Resistor SMD 0603 (1608 Metric), square (rectangular) end terminal, IPC-7351 nominal, (Body size source: IPC-SM-782 page 72, https://www.pcb-3d.com/wordpress/wp-content/uploads/ipc-sm-782a_amendment_1_and_2.pdf)")
 		(tags "resistor")
@@
 	(footprint "JST_PH_S2B-PH-K_1x02_P2.00mm_Horizontal"
 		(layer "F.Cu")
-		(at 20 80)
+		(at 100.945 -36.7)
 		(descr "JST PH series connector, S2B-PH-K (http://www.jst-mfg.com/product/pdf/eng/ePH.pdf)")
 		(tags "connector JST PH horizontal")
@@
 	(footprint "R_0603_1608Metric"
 		(layer "F.Cu")
-		(at 50 80)
+		(at 130.945 -36.7)
 		(descr "Resistor SMD 0603 (1608 Metric), square (rectangular) end terminal, IPC-7351 nominal, (Body size source: IPC-SM-782 page 72, https://www.pcb-3d.com/wordpress/wp-content/uploads/ipc-sm-782a_amendment_1_and_2.pdf)")
 		(tags "resistor")
@@
 	(footprint "C_0805_2012Metric"
 		(layer "F.Cu")
-		(at 110 20)
+		(at 220.57 -49.54)
 		(descr "Capacitor SMD 0805 (2012 Metric), square (rectangular) end terminal, IPC-7351 nominal, (Body size source: IPC-SM-782 page 76, https://www.pcb-3d.com/wordpress/wp-content/uploads/ipc-sm-782a_amendment_1_and_2.pdf, https://docs.google.com/spreadsheets/d/1BsfQQcO9C6DZCsRaXUlFlo91Tg2WpOkGARC1WS5S8t0/edit?usp=sharing)")
 		(tags "capacitor")
@@
 	(footprint "R_0603_1608Metric"
 		(layer "F.Cu")
-		(at 125 80)
+		(at 205.945 -36.7)
 		(descr "Resistor SMD 0603 (1608 Metric), square (rectangular) end terminal, IPC-7351 nominal, (Body size source: IPC-SM-782 page 72, https://www.pcb-3d.com/wordpress/wp-content/uploads/ipc-sm-782a_amendment_1_and_2.pdf)")
 		(tags "resistor")
@@
 	(footprint "SOT-23-5"
 		(layer "F.Cu")
-		(at 35 140)
+		(at 231.53 27.52)
 		(descr "SOT, 5 Pin (JEDEC MO-178 Var AA https://www.jedec.org/document_search?search_api_views_fulltext=MO-178)")
 		(tags "SOT TO_SOT_SMD")
@@
 	(footprint "R_0603_1608Metric"
 		(layer "F.Cu")
-		(at 65 80)
+		(at 145.945 -36.7)
 		(descr "Resistor SMD 0603 (1608 Metric), square (rectangular) end terminal, IPC-7351 nominal, (Body size source: IPC-SM-782 page 72, https://www.pcb-3d.com/wordpress/wp-content/uploads/ipc-sm-782a_amendment_1_and_2.pdf)")
 		(tags "resistor")
@@
 	(footprint "D_SOD-123"
 		(layer "F.Cu")
-		(at 155 20)
+		(at 35.38 25.54)
 		(descr "SOD-123")
 		(tags "SOD-123")
@@
 	(footprint "C_0805_2012Metric"
 		(layer "F.Cu")
-		(at 35 20)
+		(at 145.57 -49.54)
 		(descr "Capacitor SMD 0805 (2012 Metric), square (rectangular) end terminal, IPC-7351 nominal, (Body size source: IPC-SM-782 page 76, https://www.pcb-3d.com/wordpress/wp-content/uploads/ipc-sm-782a_amendment_1_and_2.pdf, https://docs.google.com/spreadsheets/d/1BsfQQcO9C6DZCsRaXUlFlo91Tg2WpOkGARC1WS5S8t0/edit?usp=sharing)")
 		(tags "capacitor")
@@
 	(footprint "C_0805_2012Metric"
 		(layer "F.Cu")
-		(at 95 20)
+		(at 205.57 -49.54)
 		(descr "Capacitor SMD 0805 (2012 Metric), square (rectangular) end terminal, IPC-7351 nominal, (Body size source: IPC-SM-782 page 76, https://www.pcb-3d.com/wordpress/wp-content/uploads/ipc-sm-782a_amendment_1_and_2.pdf, https://docs.google.com/spreadsheets/d/1BsfQQcO9C6DZCsRaXUlFlo91Tg2WpOkGARC1WS5S8t0/edit?usp=sharing)")
 		(tags "capacitor")
@@
 	(footprint "R_0603_1608Metric"
 		(layer "F.Cu")
-		(at 95 80)
+		(at 175.945 -36.7)
 		(descr "Resistor SMD 0603 (1608 Metric), square (rectangular) end terminal, IPC-7351 nominal, (Body size source: IPC-SM-782 page 72, https://www.pcb-3d.com/wordpress/wp-content/uploads/ipc-sm-782a_amendment_1_and_2.pdf)")
 		(tags "resistor")
@@
 	(footprint "PinHeader_1x04_P2.54mm_Vertical"
 		(layer "F.Cu")
-		(at 155 65)
+		(at 202.45 -21.56)
 		(descr "Through hole straight pin header, 1x04, 2.54mm pitch, single row")
 		(tags "Through hole pin header THT 1x04 2.54mm single row")

Commit message: Fix PCB DRC errors
Co-Authored-By: Claude Haiku 5.5 <noreply@anthropic.com>
Parts:
- C1, C2, C7, C8, C9: footprint C_0805_2012Metric -> Capacitor_SMD:C_0805_2012Metric; moved to B.Cu
- C10, C5, C6: footprint C_0603_1608Metric -> Capacitor_SMD:C_0603_1608Metric; moved to B.Cu
- D1, D10, D11, D12, D13, D14, D15, D16, D17, D18, D19, D2, D20, D21, D22, D23, D24, D25, D26, D27, D28, D29, D3, D30, D4, D5, D6, D7, D8, D9: footprint D_SOD-123 -> Diode_SMD:D_SOD-123
- J1: footprint USB_C_Receptacle_HRO_TYPE-C-31-M-12 -> Connector_USB:USB_C_Receptacle_HRO_TYPE-C-31-M-12; moved to B.Cu
- J2: footprint PinHeader_1x04_P2.54mm_Vertical -> Connector_PinHeader_2.54mm:PinHeader_1x04_P2.54mm_Vertical
- J3: footprint JST_PH_S2B-PH-K_1x02_P2.00mm_Horizontal -> Connector_JST:JST_PH_S2B-PH-K_1x02_P2.00mm_Horizontal; moved to B.Cu
- R1, R10, R2, R3, R6, R7, R8, R9: footprint R_0603_1608Metric -> Resistor_SMD:R_0603_1608Metric; moved to B.Cu
- SW1, SW10, SW11, SW12, SW13, SW14, SW15, SW16, SW17, SW18, SW19, SW2, SW20, SW21, SW22, SW23, SW24, SW25, SW26, SW27, SW28, SW29, SW3, SW30, SW4, SW5, SW6, SW7, SW8, SW9: footprint SW_Push_1TS009xxxx-xxxx-xxxx_6x6x5mm -> Button_Switch_SMD:SW_Push_1TS009xxxx-xxxx-xxxx_6x6x5mm
- SW31: footprint SW_SPDT_Shouhan_MSK12C02 -> Button_Switch_SMD:SW_SPDT_Shouhan_MSK12C02; moved to B.Cu
- U1: footprint SOIC-28W_7.5x17.9mm_P1.27mm -> Package_SO:SOIC-28W_7.5x17.9mm_P1.27mm; moved to B.Cu
- U3, U5: footprint SOT-23-5 -> Package_TO_SOT_SMD:SOT-23-5; moved to B.Cu
- U4: footprint ESP32-C3-WROOM-02U -> RF_Module:ESP32-C3-WROOM-02U; moved to B.Cu
- moved C10 244.5 mm to (70.6, 130.9)
- moved R9 231.1 mm to (47.7, 131.8), turned to -90 degrees
- moved C9 230.7 mm to (46.0, 101.3), turned to 90 degrees
- moved R10 229.8 mm to (69.4, 136.1), turned to -90 degrees
- moved U5 217.4 mm to (55.9, 97.9)
- moved U4 217.1 mm to (58.5, 135.9), turned to 180 degrees
- moved C8 215.1 mm to (44.1, 92.5)
- moved C7 213.8 mm to (65.6, 123.9), turned to 180 degrees
- moved C6 206.9 mm to (66.2, 126.2), turned to 180 degrees
- moved C5 203.3 mm to (71.7, 133.3), turned to -90 degrees
- moved R8 202.3 mm to (69.2, 124.9), turned to -90 degrees
- moved U3 193.8 mm to (50.0, 95.5), turned to 180 degrees
- moved J1 191.3 mm to (36.8, 96.3), turned to 180 degrees
- moved R6 189.3 mm to (70.1, 129.4)
- moved R7 186.7 mm to (69.3, 116.5), turned to 180 degrees
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Routing:
- net /ROW_3: track 0.00 -> 251.2 mm, vias 0 -> 1
- net GND: track 0.00 -> 192.5 mm, vias 0 -> 6
- net /ROW_2: track 0.00 -> 175.6 mm, vias 0 -> 1
- net /ROW_4: track 0.00 -> 169.1 mm, vias 0 -> 1
- net +3.3V: track 0.00 -> 120.8 mm, vias 0 -> 8
- net /ROW_1: track 0.00 -> 110.4 mm, vias 0 -> 1
- net /ROW_5: track 0.00 -> 102.3 mm, vias 0 -> 1
- net /COL_0: track 0.00 -> 97.6 mm, vias 0 -> 1
- net /COL_1: track 0.00 -> 92.9 mm, vias 0 -> 1
- net /ROW_0: track 0.00 -> 85.5 mm, vias 0 -> 1
- net /COL_2: track 0.00 -> 83.1 mm, vias 0 -> 1
- net /D-: track 0.00 -> 75.0 mm
- net /COL_4: track 0.00 -> 74.8 mm, vias 0 -> 2
- net /COL_3: track 0.00 -> 70.4 mm, vias 0 -> 1
- net /D+: track 0.00 -> 68.9 mm
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- added copper zone on B.Cu, net GND
- added copper zone on F.Cu, net GND
Other:
- board size 190 x 175 mm -> 58.2 x 69.1 mm
